File: schematic/avalon_module/avalon_module.sch (EAGLE design)
At the start: 166 parts, among them X1 332-02

Commit message: added some datasheets, updated schematic
Other:
- note added: "BUG ONLY IN DESCRIPTION ARDUINO SHIELD WITH CORRECT VOLTAGE"
Changed lines of the file:
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@@
 <text x="-881.38" y="-81.28" size="6.4516" layer="91">FIX: PLL_VOLTAGE 1V NOT 1.2V</text>
 <text x="60.96" y="-215.9" size="3.81" layer="94">CC BY-NC-SA 3.0</text>
+<text x="-881.38" y="-91.44" size="6.4516" layer="91">BUG ONLY IN DESCRIPTION ARDUINO SHIELD WITH CORRECT VOLTAGE</text>
 </plain>
 <instances>
